File: kicad/parasite.kicad_pcb (KiCad board)
At the start: 2 copper layers, 22 x 126.4 mm, 31 parts, among them Q1 MMBT3906, Q4 Q_Photo_NPN, SW1 B3U-1000P, U1 E73-2G4M08S1C, U2 SHTC3, Y1 32.768kHz

Commit message: modified PCB design for SHT4
Parts:
- U2: value SHTC3 -> SHT4x; footprint kicad:Sensirion_DFN-4-1EP_2x2mm_P1mm_EP0.7x1.6mm -> Sensor_Humidity:Sensirion_DFN-4_1.5x1.5mm_P0.8mm_SHT4x_NoCentralPad
- moved U2 0.30 mm to (73.9, 55.8)
Connections:
- U2 pad 1: +3V0 -> SDA
- U2 pad 3: SDA -> +3V0
Routing:
- net SDA: track 24.5 -> 32.6 mm
- net +3V0: track 76.5 -> 78.7 mm
