File: kicad/parasite.kicad_sch (KiCad schematic)
At the start: 29 parts, among them Q1 MMBT3906, Q4 Q_Photo_NPN, SW1 B3U-1000P, U1 E73-2G4M08S1C, U2 SHTC3, Y1 32.768kHz

Commit message: modified PCB design for SHT4
Parts:
- removed U2: SHTC3, kicad:Sensirion_DFN-4-1EP_2x2mm_P1mm_EP0.7x1.6mm, symbol Sensor_Humidity:SHTC3
- added U2: SHT4x, Sensor_Humidity:Sensirion_DFN-4_1.5x1.5mm_P0.8mm_SHT4x_NoCentralPad, symbol Sensor_Humidity:SHT4x
- RST1, SW1: DESCRIPTION Tactile Switch SPST-NO Top Actuated Surface Mount -> (none)
Connections:
- net +3V0: now also U2.3 (VDD)
- net GND: now also U2.4 (VSS)
- net SCL: now also U2.2 (SCL)
- net SDA: now also U2.1 (SDA)
